File: v1/unified/v1_unified.kicad_sch (KiCad schematic)
At the start: 193 parts, among them J1 Conn_01x01, J10 Conn_01x01, J11 Conn_01x01, J12 Conn_01x01, J13 Conn_01x01, J14 Conn_01x01, J15 Conn_01x01, J16 Conn_01x01, J17 Conn_01x01, J18 Conn_01x01, J19 Conn_01x01, J2 Conn_01x01, J20 Conn_01x01, J21 Conn_01x01, J22 Conn_01x01, J23 Conn_01x01, J24 Conn_01x01, J25 Conn_01x01, J26 Conn_01x01, J27 Conn_01x01, J28 Conn_01x01, J29 Conn_01x01, J3 Conn_01x01, J30 Conn_01x01, J31 Conn_01x01, J32 Conn_01x01, J33 Barrel_Jack, J34 Conn_01x04, J35 Conn_01x04, J36 Conn_01x04, J37 Conn_01x04, J4 Conn_01x01, J5 Conn_01x01, J6 Conn_01x01, J7 Conn_01x01, J8 Conn_01x01, J9 Conn_01x01, Q1 2N7002, Q2 2N7002, Q3 2N7002, Q4 2N7002, U1 74AHCT1G125, U2 CY8CMBR3116, U3 CY8CMBR3116

Commit message: feat: assign footprint
Parts:
- removed Q1, Q2, Q3, Q4: 2N7002, Package_TO_SOT_SMD:SOT-23, symbol Transistor_FET:2N7002
- added Q1, Q2, Q3, Q4: AO3400A, Package_TO_SOT_SMD:SOT-23, symbol Transistor_FET:AO3400A
- C1, C10, C11, C12, C13, C14, C15, C16, C17, C18, C19, C2, C20, C21, C22, C23, C24, C25, C26, C27, C28, C29, C3, C30, C31, C32, C33, C34, C35, C36, C37, C38, C39, C4, C40, C41, C42, C43, C44, C45, C46, C47, C48, C49, C5, C50, C51, C52, C53, C54, C55, C56, C58, C6, C9: footprint (none) -> Capacitor_SMD:C_0603_1608Metric
- C57: footprint (none) -> Capacitor_SMD:CP_Elec_6.3x5.4
- C7: renamed from C8; footprint (none) -> Capacitor_SMD:C_0603_1608Metric
- C8: renamed from C7; footprint (none) -> Capacitor_SMD:C_0603_1608Metric
- J34, J35, J36, J37: footprint (none) -> Connector_JST:JST_XH_B4B-XH-A_1x04_P2.50mm_Vertical
- R1, R10, R11, R12, R13, R14, R15, R16, R17, R18, R19, R2, R20, R21, R22, R23, R24, R25, R26, R27, R28, R29, R3, R30, R31, R32, R33, R34, R35, R36, R37, R38, R39, R4, R40, R41, R42, R5, R6, R7, R8, R9: footprint (none) -> Resistor_SMD:R_0603_1608Metric
- U1: footprint (none) -> Package_TO_SOT_SMD:SOT-23-5
Connections:
- net GND: now also Q1.2 (S), Q2.2 (S), Q3.2 (S), Q4.2 (S)
- net at A1.14 (GPIO10), R39.1: now also Q2.1 (G)
- net at J35.2 (Pin_2): now also Q2.3 (D)
- net at J36.2 (Pin_2): now also Q3.3 (D)
- net at A1.12 (GPIO9), R38.1: now also Q1.1 (G)
- net at A1.15 (GPIO11), R40.1: now also Q3.1 (G)
- net at A1.16 (GPIO12), R41.1: now also Q4.1 (G)
- net at J34.2 (Pin_2): now also Q1.3 (D)
- net at J37.2 (Pin_2): now also Q4.3 (D)

Commit message: feat: 0.1uF いらない
Parts:
- removed C10, C11, C12, C13, C14, C15, C16, C17, C18, C19, C20, C21, C22, C23, C24, C25, C26, C27, C28, C29, C30, C31, C32, C33, C34, C35, C36, C37, C38, C39, C40, C41, C42, C43, C44, C45, C46, C47, C48, C49, C50, C51, C52, C53, C54, C55, C56, C9: 0.1uF, Capacitor_SMD:C_0603_1608Metric, symbol Device:C

Commit message: feat: wip
Parts:
- renumbered C58 to C9, U2 to U1, U3 to U2, U1 to U3
Changed lines of the file:
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@@
 		(dnp no)
 		(fields_autoplaced yes)
-		(property "Reference" "U3"
+		(property "Reference" "U2"
 			(at 94.6719 121.92 0)
 			(show_name no)
@@
 			(project "v1_unified"
 				(path "/d245cebb-d44d-4e14-b761-281e3f34708c"
-					(reference "U3")
+					(reference "U2")
 					(unit 1)
 				)
@@
 		(dnp no)
 		(fields_autoplaced yes)
-		(property "Reference" "U1"
+		(property "Reference" "U3"
 			(at 252.73 59.8168 0)
 			(show_name no)
@@
 			(project "v1_unified"
 				(path "/d245cebb-d44d-4e14-b761-281e3f34708c"
-					(reference "U1")
+					(reference "U3")
 					(unit 1)
 				)
@@
 		(dnp no)
 		(fields_autoplaced yes)
-		(property "Reference" "U2"
+		(property "Reference" "U1"
 			(at 94.6719 39.37 0)
 			(show_name no)
@@
 			(project "v1_unified"
 				(path "/d245cebb-d44d-4e14-b761-281e3f34708c"
-					(reference "U2")
+					(reference "U1")
 					(unit 1)
 				)
@@
 		(in_pos_files yes)
 		(dnp no)
-		(property "Reference" "C58"
+		(property "Reference" "C9"
 			(at 249.174 76.708 0)
 			(show_name no)
@@
 			(project "v1_unified"
 				(path "/d245cebb-d44d-4e14-b761-281e3f34708c"
-					(reference "C58")
+					(reference "C9")
 					(unit 1)
 				)
