File: v1/slider/v1_slider.kicad_pcb (KiCad board)
At the start: 2 copper layers, 120 x 120 mm, 28 parts, among them J1 Conn_01x04, U1 CY8CMBR3108

Commit message: fix
Connections:
- E1 pad 1: /CAP1 -> /CAP0
- E2 pad 1: /CAP2 -> /CAP1
- E3 pad 1: /CAP3 -> /CAP2
- E4 pad 1: /CAP4 -> /CAP3
- E5 pad 1: /CAP5 -> /CAP4
- E6 pad 1: /CAP6 -> /CAP5
- E7 pad 1: /CAP7 -> /CAP6
- E8 pad 1: /CAP8 -> /CAP7
- R1 pad 2: /CAP1 -> /CAP0
- R2 pad 2: /CAP2 -> /CAP1
- R3 pad 2: /CAP3 -> /CAP2
- R4 pad 2: /CAP4 -> /CAP3
- R5 pad 2: /CAP5 -> /CAP4
- R6 pad 2: /CAP6 -> /CAP5
- R7 pad 2: /CAP7 -> /CAP6
- R8 pad 2: /CAP8 -> /CAP7
Changed lines of the file:
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@@
 			(layers "F.Cu")
 			(roundrect_rratio 0.02586206897)
-			(net "/CAP8")
+			(net "/CAP7")
 			(pinfunction "Pin_1_1")
 			(pintype "passive")
@@
 			(layers "F.Cu")
 			(roundrect_rratio 0.02586206897)
-			(net "/CAP2")
+			(net "/CAP1")
 			(pinfunction "Pin_1_1")
 			(pintype "passive")
@@
 			(layers "F.Cu")
 			(roundrect_rratio 0.02586206897)
-			(net "/CAP7")
+			(net "/CAP6")
 			(pinfunction "Pin_1_1")
 			(pintype "passive")
@@
 			(layers "F.Cu")
 			(roundrect_rratio 0.02586206897)
-			(net "/CAP3")
+			(net "/CAP2")
 			(pinfunction "Pin_1_1")
 			(pintype "passive")
@@
 			(layers "F.Cu")
 			(roundrect_rratio 0.02586206897)
-			(net "/CAP6")
+			(net "/CAP5")
 			(pinfunction "Pin_1_1")
 			(pintype "passive")
@@
 			(layers "F.Cu")
 			(roundrect_rratio 0.02586206897)
-			(net "/CAP1")
+			(net "/CAP0")
 			(pinfunction "Pin_1_1")
 			(pintype "passive")
@@
 			(layers "F.Cu")
 			(roundrect_rratio 0.02586206897)
-			(net "/CAP5")
+			(net "/CAP4")
 			(pinfunction "Pin_1_1")
 			(pintype "passive")
@@
 			(layers "F.Cu")
 			(roundrect_rratio 0.02586206897)
-			(net "/CAP4")
+			(net "/CAP3")
 			(pinfunction "Pin_1_1")
 			(pintype "passive")
@@
 			(layers "B.Cu" "B.Mask" "B.Paste")
 			(roundrect_rratio 0.25)
-			(net "/CAP8")
+			(net "/CAP7")
 			(pintype "passive")
 		)
@@
 			(layers "B.Cu" "B.Mask" "B.Paste")
 			(roundrect_rratio 0.25)
-			(net "/CAP7")
+			(net "/CAP6")
 			(pintype "passive")
 		)
@@
 			(layers "B.Cu" "B.Mask" "B.Paste")
 			(roundrect_rratio 0.25)
-			(net "/CAP5")
+			(net "/CAP4")
 			(pintype "passive")
 		)
@@
 			(layers "B.Cu" "B.Mask" "B.Paste")
 			(roundrect_rratio 0.25)
-			(net "/CAP3")
+			(net "/CAP2")
 			(pintype "passive")
 		)
@@
 			(layers "B.Cu" "B.Mask" "B.Paste")
 			(roundrect_rratio 0.25)
-			(net "/CAP1")
+			(net "/CAP0")
 			(pintype "passive")
 		)
@@
 			(layers "B.Cu" "B.Mask" "B.Paste")
 			(roundrect_rratio 0.25)
-			(net "/CAP6")
+			(net "/CAP5")
 			(pintype "passive")
 		)
@@
 			(layers "B.Cu" "B.Mask" "B.Paste")
 			(roundrect_rratio 0.25)
-			(net "/CAP2")
+			(net "/CAP1")
 			(pintype "passive")
 		)
@@
 			(layers "B.Cu" "B.Mask" "B.Paste")
 			(roundrect_rratio 0.25)
-			(net "/CAP4")
+			(net "/CAP3")
 			(pintype "passive")
 		)

Commit message: faet: 配線
Connections:
- R1 pad 2: /CAP0 -> /CAP6
- R2 pad 2: /CAP1 -> /CAP7
- R3 pad 2: /CAP2 -> /CAP1
- R4 pad 2: /CAP3 -> /CAP0
- R7 pad 2: /CAP6 -> /CAP3
- R8 pad 2: /CAP7 -> /CAP2
Routing:
- net /CAP1: track 0.00 -> 85.4 mm, vias 0 -> 1
- net /CAP7: track 0.00 -> 77.1 mm, vias 0 -> 1
- net /CAP3: track 0.00 -> 66.2 mm, vias 0 -> 1
- net /CAP5: track 0.00 -> 63.6 mm, vias 0 -> 1
- net /CAP0: track 0.00 -> 54.9 mm, vias 0 -> 1
- net /CAP6: track 0.00 -> 50.0 mm, vias 0 -> 1
- net /CAP4: track 0.00 -> 34.9 mm, vias 0 -> 1
- net /CAP2: track 0.00 -> 17.2 mm, vias 0 -> 1
- net /TOUCH_PWR: track 28.9 -> 46.0 mm, vias 0 -> 1
- net GND: track 0.00 -> 4.43 mm, vias 0 -> 16
- added copper zone on F.Cu, net GND

Commit message: feat: ok v1_slider
Parts:
- added H1: MountingHole, MountingHole:MountingHole_3.2mm_M3, F.Cu at (34.0, 39.0)
- added H2: MountingHole, MountingHole:MountingHole_3.2mm_M3, F.Cu at (34.0, 156.0)
- added H3: MountingHole, MountingHole:MountingHole_3.2mm_M3, F.Cu at (146.0, 39.0)
- added H4: MountingHole, MountingHole:MountingHole_3.2mm_M3, F.Cu at (146.0, 156.0)
Routing:
- net /TOUCH_PWR: track 46.0 -> 47.5 mm
- net GND: vias 16 -> 18
Other:
- board size 120 x 120 mm -> 120 x 125 mm
- board text added: "v1_slider"

Commit message: fix
Routing:
- net /CAP0: track 54.9 -> 38.6 mm
Other:
- board text added: "PWR SDA SCL GND"
Changed lines of the file:
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@@
 			)
 		)
-		(attr through_hole)
+		(attr through_hole exclude_from_pos_files exclude_from_bom)
 		(duplicate_pad_numbers_are_jumpers no)
 		(fp_line
@@
 			)
 		)
-		(attr exclude_from_bom)
+		(attr exclude_from_pos_files exclude_from_bom)
 		(duplicate_pad_numbers_are_jumpers no)
 		(fp_circle
@@
 			)
 		)
-		(attr smd)
+		(attr smd exclude_from_pos_files exclude_from_bom)
 		(duplicate_pad_numbers_are_jumpers no)
 		(fp_text user "${REFERENCE}"
@@
 			)
 		)
-		(attr smd)
+		(attr smd exclude_from_pos_files exclude_from_bom)
 		(duplicate_pad_numbers_are_jumpers no)
 		(fp_text user "${REFERENCE}"
@@
 			)
 		)
-		(attr smd)
+		(attr smd exclude_from_pos_files exclude_from_bom)
 		(duplicate_pad_numbers_are_jumpers no)
 		(fp_text user "${REFERENCE}"
@@
 			)
 		)
-		(attr through_hole)
+		(attr through_hole exclude_from_pos_files exclude_from_bom)
 		(duplicate_pad_numbers_are_jumpers no)
 		(fp_line
@@
 			)
 		)
-		(attr smd)
+		(attr smd exclude_from_pos_files exclude_from_bom)
 		(duplicate_pad_numbers_are_jumpers no)
 		(fp_text user "${REFERENCE}"
@@
 			)
 		)
-		(attr smd)
+		(attr smd exclude_from_pos_files exclude_from_bom)
 		(duplicate_pad_numbers_are_jumpers no)
 		(fp_text user "${REFERENCE}"
@@
 			)
 		)
-		(attr smd)
+		(attr smd exclude_from_pos_files exclude_from_bom)
 		(duplicate_pad_numbers_are_jumpers no)
 		(fp_text user "${REFERENCE}"
@@
 			)
 		)
-		(attr smd)
+		(attr smd exclude_from_pos_files exclude_from_bom)
 		(duplicate_pad_numbers_are_jumpers no)
 		(fp_text user "${REFERENCE}"
@@
 			)
 		)
-		(attr exclude_from_bom)
+		(attr exclude_from_pos_files exclude_from_bom)
 		(duplicate_pad_numbers_are_jumpers no)
 		(fp_circle
@@
 			)
 		)
-		(attr exclude_from_bom)
+		(attr exclude_from_pos_files exclude_from_bom)
 		(duplicate_pad_numbers_are_jumpers no)
 		(fp_circle
@@
 			)
 		)
-		(attr exclude_from_bom)
+		(attr exclude_from_pos_files exclude_from_bom)
 		(duplicate_pad_numbers_are_jumpers no)
 		(fp_circle
@@
 			)
 		)
-		(attr through_hole)
+		(attr through_hole exclude_from_pos_files exclude_from_bom)
 		(duplicate_pad_numbers_are_jumpers no)
 		(fp_line
@@
 			)
 		)
-		(attr smd)
+		(attr smd exclude_from_pos_files exclude_from_bom)
 		(duplicate_pad_numbers_are_jumpers no)
 		(fp_text user "${REFERENCE}"
@@
 		(layer "Edge.Cuts")
 	)
+	(gr_text "PWR SDA SCL GND"
+		(at 83.5 44.5 0)
+		(layer "F.SilkS")
+		(effects
+			(font
+				(size 1 1)
+				(thickness 0.1)
+			)
+			(justify left bottom)
+		)
+	)
 	(gr_text "v1_slider"
 		(at 140 58.5 0)
@@
 		(net "/CAP5")
 	)
-	(segment
-		(start 56.5 71.5)
-		(end 45 83)
-		(width 0.2)
-		(layer "F.Cu")
-		(net "/CAP0")
-	)
 	(via
