File: v1/slider/v1_slider.kicad_sch (KiCad schematic)
At the start: 0 parts

Commit message: wip
Parts:
- added C1, C3: 0.1uF, symbol Device:C
- added C2: 2.2nF, symbol Device:C
- added C4: 1uF, symbol Device:C
- added E1, E2, E3, E4, E5, E6, E7, E8: Conn_01x01, symbol Connector_Generic:Conn_01x01
- added J1: Conn_01x04, symbol Connector_Generic:Conn_01x04
- added R1, R2, R3, R4, R5, R6, R7, R8: 560, symbol Device:R
- added U1: CY8CMBR3108, Package_DFN_QFN:QFN-16-1EP_3x3mm_P0.5mm_EP1.8x1.8mm, symbol Sensor_Touch:CY8CMBR3108
Connections:
- new net: E8.1 (Pin_1), R8.1
- new net: R8.2, U1.11 (CS7)
- new net: E6.1 (Pin_1), R6.1
- new net: E4.1 (Pin_1), R4.1
- new net: R4.2, U1.13 (CS3)
- new net: E1.1 (Pin_1), R1.1
- new net: R1.2, U1.1 (CS0)
- new net: E2.1 (Pin_1), R2.1
- new net: J1.2 (Pin_2), U1.14 (SDA)
- new net: J1.3 (Pin_3), U1.15 (SCL)
- new net: E7.1 (Pin_1), R7.2
- new net: C2.1, U1.3 (CMOD)
- new net: E5.1 (Pin_1), R5.1
- new net: R5.2, U1.8 (CS4)
- new net: C1.1, U1.4 (VCC)
- new net: E3.1 (Pin_1), R3.1
- new net: R7.1, U1.10 (CS6)
- new net: R6.2, U1.9 (CS5)
- new net: R3.2, U1.12 (CS2)
- new net: R2.2, U1.2 (CS1)
- new net +5V: C3.1, C4.1, J1.4 (Pin_4), U1.5 (VDDIO), U1.6 (VDD)
- new net GND: C1.2, C2.2, C3.2, C4.2, J1.1 (Pin_1), U1.17 (EP), U1.7 (VSS)
- no-connect marks 0 -> 1

Commit message: feat: impl slider sch
Parts:
- added R10, R9: 4.7k, Resistor_SMD:R_0603_1608Metric, symbol Device:R
- C1, C2, C3, C4: footprint (none) -> Capacitor_SMD:C_0603_1608Metric
- J1: footprint (none) -> Connector_JST:JST_XH_B4B-XH-A_1x04_P2.50mm_Vertical
- R1, R2, R3, R4, R5, R6, R7, R8: footprint (none) -> Resistor_SMD:R_0603_1608Metric
Connections:
- net +5V: now also J1.1 (Pin_1), R10.1, R9.1; no longer J1.4 (Pin_4)
- net GND: now also C1.1, J1.4 (Pin_4); no longer C1.2, J1.1 (Pin_1)
- net at R8.1: now also U1.11 (CS7); no longer E8.1 (Pin_1)
- net at R8.2: now also E8.1 (Pin_1); no longer U1.11 (CS7)
- net at R6.1: now also U1.9 (CS5); no longer E6.1 (Pin_1)
- net at R4.1: now also U1.13 (CS3); no longer E4.1 (Pin_1)
- net at R4.2: now also E4.1 (Pin_1); no longer U1.13 (CS3)
- net at R1.1: now also U1.1 (CS0); no longer E1.1 (Pin_1)
- net at R1.2: now also E1.1 (Pin_1); no longer U1.1 (CS0)
- net at R2.1: now also U1.2 (CS1); no longer E2.1 (Pin_1)
- net at J1.2 (Pin_2), U1.14 (SDA): now also R9.2
- net at J1.3 (Pin_3), U1.15 (SCL): now also R10.2
- net at R5.1: now also U1.8 (CS4); no longer E5.1 (Pin_1)
- net at R5.2: now also E5.1 (Pin_1); no longer U1.8 (CS4)
- net at U1.4 (VCC): now also C1.2; no longer C1.1
- net at R3.1: now also U1.12 (CS2); no longer E3.1 (Pin_1)
- net at R6.2: now also E6.1 (Pin_1); no longer U1.9 (CS5)
- net at R3.2: now also E3.1 (Pin_1); no longer U1.12 (CS2)
- net at R2.2: now also E2.1 (Pin_1); no longer U1.2 (CS1)
Other:
- moved on the sheet: C3, C4

Commit message: fix
Parts:
- added C5: 0.1uF, Capacitor_SMD:C_0603_1608Metric, symbol Device:C
- added C6: 1uF, Capacitor_SMD:C_0603_1608Metric, symbol Device:C
- added R11, R12: 330, Resistor_SMD:R_0603_1608Metric, symbol Device:R
Connections:
- net GND: now also C5.2, C6.2
- net at J1.2 (Pin_2), R9.2: now also R11.2; no longer U1.14 (SDA)
- net at J1.3 (Pin_3), R10.2: now also R12.2; no longer U1.15 (SCL)
- net +5V renamed TOUCH_PWR
- net TOUCH_PWR: now also C5.1, C6.1
- new net: R11.1, U1.14 (SDA)
- new net: R12.1, U1.15 (SCL)

Commit message: feat: wip
Parts:
- C5: renamed from C6; value 1uF -> 0.1uF
- C6: renamed from C5; value 0.1uF -> 1uF
- E1, E2, E3, E4, E5, E6, E7, E8: footprint (none) -> v1_common:TouchPad
- R10, R9: footprint Resistor_SMD:R_0603_1608Metric -> Resistor_THT:R_Axial_DIN0207_L6.3mm_D2.5mm_P10.16mm_Horizontal
- U1: footprint Package_DFN_QFN:QFN-16-1EP_3x3mm_P0.5mm_EP1.8x1.8mm -> Package_DFN_QFN:QFN-16-1EP_3x3mm_P0.5mm_EP1.7x1.7mm
Connections:
- net CAP5: now reaches E5.1 (Pin_1), R5.2
- net CAP4: now reaches E4.1 (Pin_1), R4.2
- net CAP2: now reaches E2.1 (Pin_1), R2.2
- net CAP6: now reaches E6.1 (Pin_1), R6.2
- net CAP8: now reaches E8.1 (Pin_1), R8.2
- net CAP7: now reaches E7.1 (Pin_1), R7.2
- net CAP1: now reaches E1.1 (Pin_1), R1.2
- net CAP3: now reaches E3.1 (Pin_1), R3.2
Other:
- moved on the sheet: E1, E2, E3, E4, E5, E6, E7, E8

Commit message: fix
Connections:
- net CAP8 is gone; now on net CAP7: E8.1 (Pin_1), R8.2
- net CAP1: now also E2.1 (Pin_1), R2.2; no longer E1.1 (Pin_1), R1.2
- net CAP2: now also E3.1 (Pin_1), R3.2; no longer E2.1 (Pin_1), R2.2
- net CAP3: now also E4.1 (Pin_1), R4.2; no longer E3.1 (Pin_1), R3.2
- net CAP4: now also E5.1 (Pin_1), R5.2; no longer E4.1 (Pin_1), R4.2
- net CAP5: now also E6.1 (Pin_1), R6.2; no longer E5.1 (Pin_1), R5.2
- net CAP6: now also E7.1 (Pin_1), R7.2; no longer E6.1 (Pin_1), R6.2
- net CAP7: no longer E7.1 (Pin_1), R7.2
- new net CAP0: E1.1 (Pin_1), R1.2
Changed lines of the file:
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@@
 		)
 	)
-	(label "CAP6"
+	(label "CAP5"
 		(at 91.44 105.41 0)
 		(effects
@@
 		)
 	)
-	(label "CAP2"
+	(label "CAP1"
 		(at 91.44 95.25 0)
 		(effects
@@
 		)
 	)
-	(label "CAP7"
+	(label "CAP6"
 		(at 91.44 107.95 0)
 		(effects
@@
 		)
 	)
-	(label "CAP5"
+	(label "CAP4"
 		(at 91.44 102.87 0)
 		(effects
@@
 		)
 	)
-	(label "CAP1"
+	(label "CAP0"
 		(at 91.44 92.71 0)
 		(effects
@@
 		)
 	)
-	(label "CAP8"
+	(label "CAP7"
 		(at 91.44 110.49 0)
 		(effects
@@
 		)
 	)
-	(label "CAP4"
+	(label "CAP3"
 		(at 91.44 100.33 0)
 		(effects
@@
 		)
 	)
-	(label "CAP3"
+	(label "CAP2"
 		(at 91.44 97.79 0)
 		(effects

Commit message: faet: 配線
Connections:
- net CAP0: now also R4.2; no longer R1.2
- net CAP1: now also R3.2; no longer R2.2
- net CAP2: now also R8.2; no longer R3.2
- net CAP3: now also R7.2; no longer R4.2
- net CAP6: now also R1.2; no longer R7.2
- net CAP7: now also R2.2; no longer R8.2
Other:
- moved on the sheet: E1, E2, E3, E4, E7, E8

Commit message: feat: ok v1_slider
Parts:
- added H1, H2, H3, H4: MountingHole, MountingHole:MountingHole_3.2mm_M3, symbol Mechanical:MountingHole

Commit message: fix
Parts:
- E1, E2, E3, E4, E5, E6, E7, E8, J1, R10, R9: now left out of the parts list
Changed lines of the file:
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@@
 		(body_style 1)
 		(exclude_from_sim no)
-		(in_bom yes)
+		(in_bom no)
 		(on_board yes)
-		(in_pos_files yes)
+		(in_pos_files no)
 		(dnp no)
 		(property "Reference" "E5"
@@
 		(body_style 1)
 		(exclude_from_sim no)
-		(in_bom yes)
+		(in_bom no)
 		(on_board yes)
-		(in_pos_files yes)
+		(in_pos_files no)
 		(dnp no)
 		(property "Reference" "E4"
@@
 		(body_style 1)
 		(exclude_from_sim no)
-		(in_bom yes)
+		(in_bom no)
 		(on_board yes)
-		(in_pos_files yes)
+		(in_pos_files no)
 		(dnp no)
 		(fields_autoplaced yes)
@@
 		(in_bom no)
 		(on_board yes)
-		(in_pos_files yes)
+		(in_pos_files no)
 		(dnp no)
 		(fields_autoplaced yes)
@@
 		(body_style 1)
 		(exclude_from_sim no)
-		(in_bom yes)
+		(in_bom no)
 		(on_board yes)
-		(in_pos_files yes)
+		(in_pos_files no)
 		(dnp no)
 		(property "Reference" "E6"
@@
 		(body_style 1)
 		(exclude_from_sim no)
-		(in_bom yes)
+		(in_bom no)
 		(on_board yes)
-		(in_pos_files yes)
+		(in_pos_files no)
 		(dnp no)
 		(property "Reference" "R9"
@@
 		(body_style 1)
 		(exclude_from_sim no)
-		(in_bom yes)
+		(in_bom no)
 		(on_board yes)
-		(in_pos_files yes)
+		(in_pos_files no)
 		(dnp no)
 		(property "Reference" "E2"
@@
 		(body_style 1)
 		(exclude_from_sim no)
-		(in_bom yes)
+		(in_bom no)
 		(on_board yes)
-		(in_pos_files yes)
+		(in_pos_files no)
 		(dnp no)
 		(property "Reference" "E8"
@@
 		(body_style 1)
 		(exclude_from_sim no)
-		(in_bom yes)
+		(in_bom no)
 		(on_board yes)
-		(in_pos_files yes)
+		(in_pos_files no)
 		(dnp no)
 		(property "Reference" "E1"
@@
 		(in_bom no)
 		(on_board yes)
-		(in_pos_files yes)
+		(in_pos_files no)
 		(dnp no)
 		(fields_autoplaced yes)
@@
 		(body_style 1)
 		(exclude_from_sim no)
-		(in_bom yes)
+		(in_bom no)
 		(on_board yes)
-		(in_pos_files yes)
+		(in_pos_files no)
 		(dnp no)
 		(property "Reference" "E3"
@@
 		(body_style 1)
 		(exclude_from_sim no)
-		(in_bom yes)
+		(in_bom no)
 		(on_board yes)
-		(in_pos_files yes)
+		(in_pos_files no)
 		(dnp no)
 		(property "Reference" "R10"
@@
 		(body_style 1)
 		(exclude_from_sim no)
-		(in_bom yes)
+		(in_bom no)
 		(on_board yes)
-		(in_pos_files yes)
+		(in_pos_files no)
 		(dnp no)
 		(property "Reference" "E7"
@@
 		(in_bom no)
 		(on_board yes)
-		(in_pos_files yes)
+		(in_pos_files no)
 		(dnp no)
 		(fields_autoplaced yes)
@@
 		(in_bom no)
 		(on_board yes)
-		(in_pos_files yes)
+		(in_pos_files no)
 		(dnp no)
 		(fields_autoplaced yes)
