File: v1/pcb/v1.kicad_pcb (KiCad board)
At the start: 2 copper layers, 120 x 125 mm, 32 parts, among them J1 Conn_01x04, U1 CY8CMBR3108

Commit message: refactor: organize PCB and firmware by revision
Other:
- board text added: "v1"
- board text removed: "v1_slider"
Changed lines of the file:
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@@
 		(property ki_fp_filters "Connector*:*_1x??_*")
 		(sheetname "/")
-		(sheetfile "v1_slider.kicad_sch")
+		(sheetfile "v1.kicad_sch")
 		(units
 			(unit
@@
 		(property ki_fp_filters "MountingHole*")
 		(sheetname "/")
-		(sheetfile "v1_slider.kicad_sch")
+		(sheetfile "v1.kicad_sch")
 		(units
 			(unit
@@
 		(property ki_fp_filters "Connector*:*_1x??_*")
 		(sheetname "/")
-		(sheetfile "v1_slider.kicad_sch")
+		(sheetfile "v1.kicad_sch")
 		(units
 			(unit
@@
 		(property ki_fp_filters "Connector*:*_1x??_*")
 		(sheetname "/")
-		(sheetfile "v1_slider.kicad_sch")
+		(sheetfile "v1.kicad_sch")
 		(units
 			(unit
@@
 		(property ki_fp_filters "Connector*:*_1x??_*")
 		(sheetname "/")
-		(sheetfile "v1_slider.kicad_sch")
+		(sheetfile "v1.kicad_sch")
 		(units
 			(unit
@@
 		(property ki_fp_filters "R_*")
 		(sheetname "/")
-		(sheetfile "v1_slider.kicad_sch")
+		(sheetfile "v1.kicad_sch")
 		(units
 			(unit
@@
 		(property ki_fp_filters "Connector*:*_1x??_*")
 		(sheetname "/")
-		(sheetfile "v1_slider.kicad_sch")
+		(sheetfile "v1.kicad_sch")
 		(units
 			(unit
@@
 		(property ki_fp_filters "Connector*:*_1x??_*")
 		(sheetname "/")
-		(sheetfile "v1_slider.kicad_sch")
+		(sheetfile "v1.kicad_sch")
 		(units
 			(unit
@@
 		(property ki_fp_filters "Connector*:*_1x??_*")
 		(sheetname "/")
-		(sheetfile "v1_slider.kicad_sch")
+		(sheetfile "v1.kicad_sch")
 		(units
 			(unit
@@
 		(property ki_fp_filters "Connector*:*_1x??_*")
 		(sheetname "/")
-		(sheetfile "v1_slider.kicad_sch")
+		(sheetfile "v1.kicad_sch")
 		(units
 			(unit
@@
 		(property ki_fp_filters "MountingHole*")
 		(sheetname "/")
-		(sheetfile "v1_slider.kicad_sch")
+		(sheetfile "v1.kicad_sch")
 		(units
 			(unit
@@
 		(property ki_fp_filters "MountingHole*")
 		(sheetname "/")
-		(sheetfile "v1_slider.kicad_sch")
+		(sheetfile "v1.kicad_sch")
 		(units
 			(unit
@@
 		(property ki_fp_filters "MountingHole*")
 		(sheetname "/")
-		(sheetfile "v1_slider.kicad_sch")
+		(sheetfile "v1.kicad_sch")
 		(units
 			(unit
@@
 		(property ki_fp_filters "R_*")
 		(sheetname "/")
-		(sheetfile "v1_slider.kicad_sch")
+		(sheetfile "v1.kicad_sch")
 		(units
 			(unit
@@
 		(property ki_fp_filters "Connector*:*_1x??_*")
 		(sheetname "/")
-		(sheetfile "v1_slider.kicad_sch")
+		(sheetfile "v1.kicad_sch")
 		(units
 			(unit
@@
 		(property ki_fp_filters "R_*")
 		(sheetname "/")
-		(sheetfile "v1_slider.kicad_sch")
+		(sheetfile "v1.kicad_sch")
 		(units
 			(unit
@@
 		(property ki_fp_filters "QFN*1EP*3x3mm*P0.5mm*")
 		(sheetname "/")
-		(sheetfile "v1_slider.kicad_sch")
+		(sheetfile "v1.kicad_sch")
 		(units
 			(unit
@@
 		(property ki_fp_filters "R_*")
 		(sheetname "/")
-		(sheetfile "v1_slider.kicad_sch")
+		(sheetfile "v1.kicad_sch")
 		(units
 			(unit
@@
 		(property ki_fp_filters "R_*")
 		(sheetname "/")
-		(sheetfile "v1_slider.kicad_sch")
+		(sheetfile "v1.kicad_sch")
 		(units
 			(unit
@@
 		(property ki_fp_filters "C_*")
 		(sheetname "/")
-		(sheetfile "v1_slider.kicad_sch")
+		(sheetfile "v1.kicad_sch")
 		(units
 			(unit
@@
 		(property ki_fp_filters "R_*")
 		(sheetname "/")
-		(sheetfile "v1_slider.kicad_sch")
+		(sheetfile "v1.kicad_sch")
 		(units
 			(unit
@@
 		(property ki_fp_filters "C_*")
 		(sheetname "/")
-		(sheetfile "v1_slider.kicad_sch")
+		(sheetfile "v1.kicad_sch")
 		(units
 			(unit
@@
 		(property ki_fp_filters "R_*")
 		(sheetname "/")
-		(sheetfile "v1_slider.kicad_sch")
+		(sheetfile "v1.kicad_sch")
 		(units
 			(unit
@@
 		(property ki_fp_filters "C_*")
 		(sheetname "/")
-		(sheetfile "v1_slider.kicad_sch")
+		(sheetfile "v1.kicad_sch")
 		(units
 			(unit
@@
 		(property ki_fp_filters "C_*")
 		(sheetname "/")
-		(sheetfile "v1_slider.kicad_sch")
+		(sheetfile "v1.kicad_sch")
 		(units
 			(unit
@@
 		(property ki_fp_filters "R_*")
 		(sheetname "/")
-		(sheetfile "v1_slider.kicad_sch")
+		(sheetfile "v1.kicad_sch")
 		(units
 			(unit
@@
 		(property ki_fp_filters "R_*")
 		(sheetname "/")
-		(sheetfile "v1_slider.kicad_sch")
+		(sheetfile "v1.kicad_sch")
 		(units
 			(unit
@@
 		(property ki_fp_filters "R_*")
 		(sheetname "/")
-		(sheetfile "v1_slider.kicad_sch")
+		(sheetfile "v1.kicad_sch")
 		(units
 			(unit
@@
 		(property ki_fp_filters "R_*")
 		(sheetname "/")
-		(sheetfile "v1_slider.kicad_sch")
+		(sheetfile "v1.kicad_sch")
 		(units
 			(unit
@@
 		(property ki_fp_filters "R_*")
 		(sheetname "/")
-		(sheetfile "v1_slider.kicad_sch")
+		(sheetfile "v1.kicad_sch")
 		(units
 			(unit
@@
 		(property ki_fp_filters "C_*")
 		(sheetname "/")
-		(sheetfile "v1_slider.kicad_sch")
+		(sheetfile "v1.kicad_sch")
 		(units
 			(unit
@@
 		(property ki_fp_filters "C_*")
 		(sheetname "/")
-		(sheetfile "v1_slider.kicad_sch")
+		(sheetfile "v1.kicad_sch")
 		(units
 			(unit
@@
 		)
 	)
-	(gr_text "v1_slider"
+	(gr_text "v1"
 		(at 140 58.5 0)
 		(layer "F.SilkS")
